Commit message: Further renaming

File: urdf/scout_v2.urdf (robot description, URDF)
Before this commit: robot scout_v2, 7 links, 6 joints
Links:
- link base_link: geometry collision box size=0.15416666666666667 0.627 0.06999999999999999; collision box size=0.925 0.38 0.21
- link front_left_wheel_link: geometry collision cylinder length=0.11653 radius=0.16459; visual mesh filename=package://nav2_tutorial/meshes/scout_v2/wheel_type2.dae
- link front_right_wheel_link: geometry collision cylinder length=0.11653 radius=0.16459; visual mesh filename=package://nav2_tutorial/meshes/scout_v2/wheel_type1.dae
- link rear_left_wheel_link: geometry collision cylinder length=0.11653 radius=0.16459; visual mesh filename=package://nav2_tutorial/meshes/scout_v2/wheel_type1.dae
- link rear_right_wheel_link: geometry collision cylinder length=0.11653 radius=0.16459; visual mesh filename=package://nav2_tutorial/meshes/scout_v2/wheel_type2.dae

File: urdf/scout_v2.xacro (robot description, xacro)
@@ -3,6 +3,6 @@
     xmlns:xacro="http://ros.org/wiki/xacro">
     <xacro:arg name="robot_namespace" default="/" />
-    <xacro:include filename="$(find agilex_demo)/urdf/scout_wheel_type1.xacro" />
-    <xacro:include filename="$(find agilex_demo)/urdf/scout_wheel_type2.xacro" />
+    <xacro:include filename="$(find nav2_tutorial)/urdf/scout_wheel_type1.xacro" />
+    <xacro:include filename="$(find nav2_tutorial)/urdf/scout_wheel_type2.xacro" />
     <!-- Variables -->
     <xacro:property name="M_PI" value="3.14159"/>
@@ -21,5 +21,5 @@
             <origin xyz="0 0 0" rpy="0 0 0" />
             <geometry>
-                <mesh filename="package://agilex_demo/meshes/scout_v2/base_link.dae" />
+                <mesh filename="package://nav2_tutorial/meshes/scout_v2/base_link.dae" />
             </geometry>
         </visual>

File: urdf/scout_vrtk.urdf (robot description, URDF)
Before this commit: robot scout_vrtk, 9 links, 8 joints
Links:
- link base_link: geometry collision box size=0.15416666666666667 0.627 0.06999999999999999; collision box size=0.925 0.38 0.21
- link front_left_wheel_link: geometry collision cylinder length=0.11653 radius=0.16459; visual mesh filename=package://nav2_tutorial/meshes/scout_v2/wheel_type2.dae
- link front_right_wheel_link: geometry collision cylinder length=0.11653 radius=0.16459; visual mesh filename=package://nav2_tutorial/meshes/scout_v2/wheel_type1.dae
- link rear_left_wheel_link: geometry collision cylinder length=0.11653 radius=0.16459; visual mesh filename=package://nav2_tutorial/meshes/scout_v2/wheel_type1.dae
- link rear_right_wheel_link: geometry collision cylinder length=0.11653 radius=0.16459; visual mesh filename=package://nav2_tutorial/meshes/scout_v2/wheel_type2.dae

File: urdf/scout_vrtk.xacro (robot description, xacro)
@@ -2,5 +2,5 @@
 <robot name="scout_vrtk"
     xmlns:xacro="http://ros.org/wiki/xacro">
-    <xacro:include filename="$(find agilex_demo)/urdf/scout_v2.xacro" />
+    <xacro:include filename="$(find nav2_tutorial)/urdf/scout_v2.xacro" />
     <!-- For testing, hang the robot up in the air -->
     <!-- <link name="world" />

File: urdf/scout_wheel_type1.xacro (robot description, xacro)
@@ -34,5 +34,5 @@
                 <origin xyz="0 0 0" rpy="0 0 0" />
                 <geometry>
-                    <mesh filename="package://agilex_demo/meshes/scout_v2/wheel_type1.dae" />
+                    <mesh filename="package://nav2_tutorial/meshes/scout_v2/wheel_type1.dae" />
                 </geometry>
             </visual>

File: urdf/scout_wheel_type2.xacro (robot description, xacro)
@@ -34,5 +34,5 @@
                 <origin xyz="0 0 0" rpy="0 0 0" />
                 <geometry>
-                    <mesh filename="package://agilex_demo/meshes/scout_v2/wheel_type2.dae" />
+                    <mesh filename="package://nav2_tutorial/meshes/scout_v2/wheel_type2.dae" />
                 </geometry>
             </visual>
